File: Hardware/Qwiic 1x1/SparkFun_Qwiic_Accelerometer_BMA400.brd (EAGLE design)
At the start: 25.4 x 25.4 mm, 56 parts, among them J1 QWIIC_RIGHT_ANGLE, J2 QWIIC_RIGHT_ANGLE, U1 BMA400

Commit message: Change default I2C address
Parts:
- turned ADR to 180 degrees
Connections:
- net N$5: now also ADR.1; no longer ADR.3
- net N$6: now also ADR.3; no longer ADR.1
Changed lines of the file:
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@@
 <attribute name="VALUE" x="8.89" y="16.002" size="0.6096" layer="27" font="vector" ratio="20" rot="R180" align="top-center"/>
-</element>
-<element name="ADR" library="SparkFun-Jumpers" package="SMT-JUMPER_3_1-NC_TRACE_SILK" package3d_urn="urn:adsk.eagle:package:39288/1" value="JUMPER-SMT_3_1-NC_TRACE_SILK" x="12.7" y="15.24" smashed="yes" rot="MR0">
-<attribute name="NAME" x="12.7" y="16.383" size="0.6096" layer="26" font="vector" ratio="20" rot="MR0" align="bottom-center"/>
-<attribute name="VALUE" x="12.7" y="14.097" size="0.6096" layer="28" font="vector" ratio="20" rot="MR0" align="top-center"/>
 </element>
 <element name="U$1" library="output" package="PWR0" value="" x="22.86" y="20.32" smashed="yes"/>
@@
 <element name="U$6" library="output" package="#_3V3#6" value="" x="8.89" y="1.27" smashed="yes" rot="R90"/>
 <element name="U$28" library="output" package="#_GND#6" value="" x="6.35" y="1.27" smashed="yes" rot="R90"/>
+<element name="ADR" library="SparkFun-Jumpers" package="SMT-JUMPER_3_1-NC_TRACE_SILK" package3d_urn="urn:adsk.eagle:package:39288/1" value="JUMPER-SMT_3_1-NC_TRACE_SILK" x="12.7" y="15.24" smashed="yes" rot="MR180">
+<attribute name="NAME" x="12.7" y="14.097" size="0.6096" layer="26" font="vector" ratio="20" rot="MR180" align="bottom-center"/>
+<attribute name="VALUE" x="12.7" y="16.383" size="0.6096" layer="28" font="vector" ratio="20" rot="MR180" align="top-center"/>
+</element>
 </elements>
 <signals>
@@
 <contactref element="U1" pad="1"/>
 <contactref element="J3" pad="5"/>
-<contactref element="ADR" pad="2"/>
 <wire x1="16.51" y1="7.366" x2="16.51" y2="1.27" width="0.2032" layer="1"/>
 <wire x1="13.475" y1="11.95" x2="14.11189375" y2="11.95" width="0.2032" layer="1"/>
@@
 <wire x1="16.51" y1="7.366" x2="13.475" y2="10.401" width="0.2032" layer="1"/>
 <wire x1="13.475" y1="10.401" x2="13.475" y2="11.95" width="0.2032" layer="1"/>
+<contactref element="ADR" pad="2"/>
 </signal>
 <signal name="!CS!">
@@
 <signal name="N$5">
 <contactref element="R5" pad="1"/>
-<contactref element="ADR" pad="3"/>
 <wire x1="9.74" y1="15.24" x2="10.8204" y2="15.24" width="0.2032" layer="1"/>
 <via x="10.8204" y="15.24" extent="1-16" drill="0.3048"/>
 <wire x1="10.8204" y1="15.24" x2="11.6586" y2="15.24" width="0.2032" layer="16"/>
+<contactref element="ADR" pad="1"/>
 </signal>
 <signal name="N$6">
 <contactref element="R4" pad="2"/>
-<contactref element="ADR" pad="1"/>
 <wire x1="13.7414" y1="15.24" x2="14.5796" y2="15.24" width="0.2032" layer="16"/>
 <via x="14.5796" y="15.24" extent="1-16" drill="0.3048"/>
 <wire x1="14.5796" y1="15.24" x2="15.66" y2="15.24" width="0.2032" layer="1"/>
+<contactref element="ADR" pad="3"/>
 </signal>
 <signal name="N$1">
