File: Hardware/Qwiic 1x1/SparkFun_Qwiic_Accelerometer_BMA400.sch (EAGLE design)
At the start: 30 parts, among them J1 QWIIC_RIGHT_ANGLE, J2 QWIIC_RIGHT_ANGLE, U1 BMA400

Commit message: Update version number to v10
Other:
- note added: "v10"
- note removed: "v01"
Changed lines of the file:
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@@
 <plain>
 <text x="167.64" y="10.16" size="2.54" layer="94" font="vector">Dryw Wade</text>
-<text x="238.76" y="7.62" size="2.54" layer="94" font="vector">v01</text>
+<text x="238.76" y="7.62" size="2.54" layer="94" font="vector">v10</text>
 <text x="73.66" y="180.34" size="2.54" layer="94" font="vector" align="center">Accelerometer - BMA400</text>
 <text x="38.1" y="76.2" size="2.54" layer="94" font="vector" align="center">Connectors</text>

Commit message: Remove library file
Part is in SFE Eagle library, update part in design
Parts:
- U1: device BMA400:BMA400 -> SparkFun-Sensors:BMA400
Changed lines of the file:
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@@
 <parts>
 <part name="FRAME1" library="SparkFun-Aesthetics" deviceset="FRAME-LETTER" device=""/>
-<part name="U1" library="BMA400" deviceset="BMA400" device=""/>
+<part name="U1" library="SparkFun-Sensors" deviceset="BMA400" device=""/>
 <part name="LOGO1" library="SparkFun-Aesthetics" deviceset="QWIIC_LOGO" device="_5MM"/>
 <part name="J1" library="SparkFun-Connectors" deviceset="QWIIC_CONNECTOR" device="JS-1MM" value="QWIIC_RIGHT_ANGLE"/>
